File: PCB/numberpad.kicad_pcb (KiCad board)
At the start: 2 copper layers, 97 x 127.2 mm, 73 parts, among them J1 Light_Sensor, J2 Rotary_Encoder, J3 Screen_Connector, J4 FingerPrint_UART, J5 USB_A, J6 Programmer, J7 USB_C_TO_PC, SW0 0, SW1 ., SW10 8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

Commit message: jlcpcb update
Routing:
- net DS-: track 79.2 -> 71.0 mm
- net C1: track 130.2 -> 125.5 mm
- net DT: track 85.5 -> 81.2 mm, vias 1 -> 0
- net CLK: track 78.0 -> 75.7 mm
- net C0: track 118.7 -> 116.8 mm
- net SCREEN_CS: track 56.9 -> 58.2 mm
- net R3_LED: track 88.9 -> 90.0 mm
- net Net-(D17-DOUT): track 29.1 -> 28.1 mm
- net R1_LED: track 98.7 -> 97.7 mm
- net Net-(D23-DOUT): track 15.6 -> 14.7 mm
- net Net-(D32-DOUT): track 14.0 -> 13.2 mm
- net Net-(D21-DOUT): track 22.6 -> 21.9 mm
- net Net-(D30-DOUT): track 15.1 -> 14.4 mm
- net R3: track 182.0 -> 181.4 mm
- net Net-(D24-DOUT): track 15.5 -> 14.8 mm
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